File: kicadFiles/arcticPCB.sch (KiCad schematic (older format))
At the start: 175 parts, among them J1 TYPE-C-31-M12_13, J2 Conn_01x14, J3 Conn_ARM_JTAG_SWD_10, SW1 ESC, SW10 9, SW11 0, SW12 -_, SW13 +=, SW14 2U BKSP, SW15 TAB_150, SW16 Q, SW17 W, SW18 E, SW19 R, SW2 1, SW20 T, SW21 Y, SW22 U, SW23 I, SW24 O, SW25 P, SW26 [{, SW27 ]}, SW28 \\|_150, SW29 CAPS_175, SW3 2, SW30 A, SW31 S, SW32 D, SW33 F, SW34 G, SW35 H, SW36 J, SW37 K, SW38 L, SW39 :;, SW4 3, SW40 \"', SW41 ENTER_225, SW42 LSHIFT_225, SW43 Z, SW44 X, SW45 C, SW46 V, SW47 B, SW48 N, SW49 M, SW5 4, SW50 <,, SW51 >., SW52 ?/, SW53 RSHIFT_275, SW54 LCTRL_150, SW55 LGUI_100, SW56 LALT_150, SW57 SPACE_7U, SW58 RALT_150, SW59 RGUI_100, SW6 5, SW60 RCTRL_150, SW61 FN_100, SW62 RSHIFT_175, SW63 STEPPED_CAPS_125, SW64 1U LBKSP, SW65 1U RBKSP, SW7 6, SW8 7, SW9 8, U1 STM32F072-LQFP48, U2 USBLC6-2SC6, U3 MCP1700-3302E_SOT23

Commit message: Working with standard Kicad
Parts:
- CB1, CB2, CB3, CB4, CB5, CB6, CB7, CB8, CRST1, CRST2, CSH1, CSH2, CSI1, CSO1, CUSB1: symbol Device:C_Small -> arcticPCB-rescue:C_Small-Device
- D1, D10, D11, D12, D13, D14, D15, D16, D17, D18, D19, D2, D20, D21, D22, D23, D24, D25, D26, D27, D28, D29, D3, D30, D31, D32, D33, D34, D35, D36, D37, D38, D39, D4, D40, D41, D42, D43, D44, D45, D46, D47, D48, D49, D5, D50, D51, D52, D53, D54, D55, D56, D57, D58, D59, D6, D60, D62, D65, D7, D8, D9, DRST1, DS1, DSH1: symbol Device:D -> arcticPCB-rescue:D-Device
- DF1: symbol Device:D_Schottky -> arcticPCB-rescue:D_Schottky-Device
- F1: symbol Device:Polyfuse_Small -> arcticPCB-rescue:Polyfuse_Small-Device
- H1, H10, H2, H3, H4, H5, H6, H7, H9, L1, L2, L3, L4, L5: symbol Mechanical:MountingHole -> arcticPCB-rescue:MountingHole-Mechanical
- H8: symbol Mechanical:MountingHole_Pad -> arcticPCB-rescue:MountingHole_Pad-Mechanical
- J2: symbol Connector_Generic:Conn_01x14 -> arcticPCB-rescue:Conn_01x14-Connector_Generic
- J3: symbol Connector:Conn_ARM_JTAG_SWD_10 -> arcticPCB-rescue:Conn_ARM_JTAG_SWD_10-Connector
- QRST1: symbol Transistor_BJT:DTC123J -> arcticPCB-rescue:DTC123J-Transistor_BJT
- RCC1, RCC2, RRST1, RSH1, RSH2: symbol Device:R_Small -> arcticPCB-rescue:R_Small-Device
- SWRST1: symbol Switch:SW_Push -> arcticPCB-rescue:SW_Push-Switch
- U2: symbol Power_Protection:USBLC6-2SC6 -> arcticPCB-rescue:USBLC6-2SC6-Power_Protection
